File: extras/basic_circuit.sch (EAGLE design)
At the start: 15 parts, among them M1 ARDUINO-PRO-MINI-3.3V, U1 SI4703

Commit message: SI4703 Arduino Library
Parts:
- added CX1, CX2: (no value), rcl:CXXC10B6
- added J1: (no value), SparkFun-Connectors:AUDIO_JACK_2.5MM_HOLESONLY
Connections:
- new net N$16: CX1.1, U1.ROUT
- new net N$19: CX2.1, U1.LOUT
- new net N$20: CX1.2, J1.RIGHT
- new net N$21: CX2.2, J1.LEFT
- net GND: now also J1.SLEEVE
Changed lines of the file:
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@@
 <?xml version="1.0" encoding="utf-8"?>
 <!DOCTYPE eagle SYSTEM "eagle.dtd">
-<eagle version="9.4.2">
+<eagle version="9.6.2">
 <drawing>
 <settings>
@@
 <layer number="112" name="tSilk" color="7" fill="1" visible="no" active="yes"/>
 <layer number="113" name="ReferenceLS" color="7" fill="1" visible="no" active="no"/>
+<layer number="114" name="Badge_Outline" color="7" fill="1" visible="yes" active="yes"/>
+<layer number="115" name="ReferenceISLANDS" color="7" fill="1" visible="yes" active="yes"/>
 <layer number="116" name="Patch_BOT" color="9" fill="4" visible="no" active="yes"/>
 <layer number="118" name="Rect_Pads" color="7" fill="1" visible="no" active="no"/>
@@
 <part name="R2" library="SparkFun-Resistors" library_urn="urn:adsk.eagle:library:532" deviceset="4.7KOHM" device="-0603-1/10W-1%" package3d_urn="urn:adsk.eagle:package:39650/1" value="4.7k"/>
 <part name="SUPPLY5" library="supply2" library_urn="urn:adsk.eagle:library:372" deviceset="VCC" device=""/>
+<part name="J1" library="SparkFun-Connectors" library_urn="urn:adsk.eagle:library:513" deviceset="AUDIO_JACK_2.5MM" device="_HOLESONLY" package3d_urn="urn:adsk.eagle:package:37993/1"/>
+<part name="CX1" library="rcl" library_urn="urn:adsk.eagle:library:334" deviceset="CX" device="XC10B6" package3d_urn="urn:adsk.eagle:package:23700/1"/>
+<part name="CX2" library="rcl" library_urn="urn:adsk.eagle:library:334" deviceset="CX" device="XC10B6" package3d_urn="urn:adsk.eagle:package:23700/1"/>
 </parts>
 <sheets>
@@
 <attribute name="VALUE" x="51.435" y="104.775" size="1.778" layer="96"/>
 </instance>
+<instance part="J1" gate="G$1" x="127" y="45.72" smashed="yes" rot="R90">
+<attribute name="NAME" x="123.952" y="40.64" size="1.778" layer="95" font="vector" rot="R90"/>
+<attribute name="VALUE" x="132.08" y="40.64" size="1.778" layer="96" font="vector" rot="R90"/>
+</instance>
+<instance part="CX1" gate="G$1" x="121.92" y="60.96" smashed="yes">
+<attribute name="NAME" x="123.444" y="61.341" size="1.778" layer="95"/>
+<attribute name="VALUE" x="123.444" y="56.261" size="1.778" layer="96"/>
+</instance>
+<instance part="CX2" gate="G$1" x="132.08" y="60.96" smashed="yes">
+<attribute name="NAME" x="133.604" y="61.341" size="1.778" layer="95"/>
+<attribute name="VALUE" x="133.604" y="56.261" size="1.778" layer="96"/>
+</instance>
 </instances>
 <busses>
@@
 <pinref part="GND1" gate="1" pin="GND"/>
 <wire x1="111.76" y1="58.42" x2="111.76" y2="53.34" width="0.1524" layer="91"/>
+<pinref part="J1" gate="G$1" pin="SLEEVE"/>
+<wire x1="124.46" y1="50.8" x2="124.46" y2="53.34" width="0.1524" layer="91"/>
+<wire x1="124.46" y1="53.34" x2="111.76" y2="53.34" width="0.1524" layer="91"/>
+<junction x="111.76" y="53.34"/>
 </segment>
 <segment>
@@
 </segment>
 </net>
+<net name="N$16" class="0">
+<segment>
+<pinref part="U1" gate="G$1" pin="ROUT"/>
+<pinref part="CX1" gate="G$1" pin="1"/>
+<wire x1="116.84" y1="68.58" x2="121.92" y2="68.58" width="0.1524" layer="91"/>
+<wire x1="121.92" y1="68.58" x2="121.92" y2="63.5" width="0.1524" layer="91"/>
+</segment>
+</net>
+<net name="N$19" class="0">
+<segment>
+<pinref part="U1" gate="G$1" pin="LOUT"/>
+<pinref part="CX2" gate="G$1" pin="1"/>
+<wire x1="116.84" y1="71.12" x2="132.08" y2="71.12" width="0.1524" layer="91"/>
+<wire x1="132.08" y1="71.12" x2="132.08" y2="63.5" width="0.1524" layer="91"/>
+</segment>
+</net>
+<net name="N$20" class="0">
+<segment>
+<pinref part="J1" gate="G$1" pin="RIGHT"/>
+<wire x1="127" y1="50.8" x2="127" y2="55.88" width="0.1524" layer="91"/>
+<pinref part="CX1" gate="G$1" pin="2"/>
+<wire x1="127" y1="55.88" x2="121.92" y2="55.88" width="0.1524" layer="91"/>
+</segment>
+</net>
+<net name="N$21" class="0">
+<segment>
+<pinref part="J1" gate="G$1" pin="LEFT"/>
+<pinref part="CX2" gate="G$1" pin="2"/>
+<wire x1="129.54" y1="50.8" x2="129.54" y2="55.88" width="0.1524" layer="91"/>
+<wire x1="129.54" y1="55.88" x2="132.08" y2="55.88" width="0.1524" layer="91"/>
+</segment>
+</net>
