File: extras/schematic/basic_attiny84.sch (EAGLE design)
At the start: 14 parts, among them U1 SI4703

Commit message: SI470X Arduino Library
Other:
- note added: "Not necessary if you are using module"
Changed lines of the file:
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@@
 <drawing>
 <settings>
-<setting alwaysvectorfont="yes"/>
+<setting alwaysvectorfont="no"/>
 <setting verticaltext="up"/>
 </settings>
@@
 <layer number="155" name="FabDoc3" color="7" fill="15" visible="no" active="no"/>
 <layer number="199" name="Contour" color="7" fill="1" visible="no" active="yes"/>
-<layer number="200" name="200bmp" color="1" fill="10" visible="no" active="yes"/>
+<layer number="200" name="200bmp" color="1" fill="10" visible="yes" active="yes"/>
 <layer number="201" name="201bmp" color="2" fill="1" visible="no" active="no"/>
 <layer number="202" name="202bmp" color="3" fill="1" visible="no" active="no"/>
@@
 <sheet>
 <plain>
+<rectangle x1="35.56" y1="88.9" x2="73.66" y2="111.76" layer="200"/>
+<text x="33.02" y="114.3" size="1.778" layer="200">Not necessary if you are using module</text>
+<rectangle x1="68.58" y1="35.56" x2="91.44" y2="58.42" layer="200"/>
+<rectangle x1="119.38" y1="55.88" x2="139.7" y2="76.2" layer="200"/>
 </plain>
 <instances>
