File: extras/schematic/basic_attiny85.sch (EAGLE design)
At the start: 13 parts, among them U1 SI4703, U2 ATTINY85-20P

Commit message: SI470X Arduino Library
Other:
- note added: "Not necessary if you are using module"
Changed lines of the file:
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@@
 <drawing>
 <settings>
-<setting alwaysvectorfont="yes"/>
+<setting alwaysvectorfont="no"/>
 <setting verticaltext="up"/>
 </settings>
@@
 <layer number="155" name="FabDoc3" color="7" fill="15" visible="no" active="no"/>
 <layer number="199" name="Contour" color="7" fill="1" visible="no" active="yes"/>
-<layer number="200" name="200bmp" color="1" fill="10" visible="no" active="yes"/>
+<layer number="200" name="200bmp" color="1" fill="10" visible="yes" active="yes"/>
 <layer number="201" name="201bmp" color="2" fill="1" visible="no" active="no"/>
 <layer number="202" name="202bmp" color="3" fill="1" visible="no" active="no"/>
@@
 <sheet>
 <plain>
+<rectangle x1="40.64" y1="88.9" x2="66.04" y2="106.68" layer="200"/>
+<rectangle x1="68.58" y1="33.02" x2="91.44" y2="58.42" layer="200"/>
+<rectangle x1="116.84" y1="55.88" x2="139.7" y2="73.66" layer="200"/>
+<text x="33.02" y="109.22" size="1.778" layer="200">Not necessary if you are using module</text>
 </plain>
 <instances>
